Commit message: 更新配置文件

File: src/dummy_rtx_description/urdf/dummy_ros_r.xacro (robot description, xacro)
@@ -1,36 +1,27 @@
 <?xml version="1.0" ?>
 <robot name="dummy_ros_r" xmlns:xacro="http://www.ros.org/wiki/xacro">
-  <!-- 引入 xacro 子模块 -->
-  <xacro:include filename="$(find dummy_ros_r_description)/urdf/materials.xacro" />
-  <xacro:include filename="$(find dummy_ros_r_description)/urdf/dummy_ros_r.trans" />
-  <xacro:include filename="$(find dummy_ros_r_description)/urdf/dummy_ros_r.gazebo" />
-  <!-- ✅ 添加 dummy 根 link 和 fixed joint -->
-  <link name="base_dummy"/>
-  <joint name="fixed_base_to_real_base" type="fixed">
-    <parent link="base_dummy"/>
-    <child link="base_link"/>
+<xacro:include filename="$(find dummy_rtx_description)/urdf/materials.xacro" />
+<xacro:include filename="$(find dummy_rtx_description)/urdf/dummy_ros_r.trans" />
+<xacro:include filename="$(find dummy_rtx_description)/urdf/dummy_ros_r.gazebo" />
+<link name="base_link">
+  <inertial>
+    <origin xyz="-1.6917018154750703e-07 -0.003158223450406361 0.04988890332172506" rpy="0 0 0"/>
+    <mass value="1.0265532197281713"/>
+    <inertia ixx="0.002" iyy="0.002095" izz="0.001994" ixy="0.0" iyz="1.5e-05" ixz="0.0"/>
+  </inertial>
+  <visual>
     <origin xyz="0 0 0" rpy="0 0 0"/>
-  </joint>
-  <!-- ✅ 原始 base_link 开始 -->
-  <link name="base_link">
-    <inertial>
-      <origin xyz="-1.6917018154750703e-07 -0.003158223450406361 0.04988890332172506" rpy="0 0 0"/>
-      <mass value="1.0265532197281713"/>
-      <inertia ixx="0.002" iyy="0.002095" izz="0.001994" ixy="0.0" iyz="1.5e-05" ixz="0.0"/>
-    </inertial>
-    <visual>
-      <origin xyz="0 0 0" rpy="0 0 0"/>
-      <geometry>
-        <mesh filename="file://$(find dummy_ros_r_description)/meshes/base_link.stl" scale="0.001 0.001 0.001"/>
-      </geometry>
-      <material name="silver"/>
-    </visual>
-    <collision>
-      <origin xyz="0 0 0" rpy="0 0 0"/>
-      <geometry>
-        <mesh filename="file://$(find dummy_ros_r_description)/meshes/base_link.stl" scale="0.001 0.001 0.001"/>
-      </geometry>
-    </collision>
-  </link>
+    <geometry>
+      <mesh filename="file://$(find dummy_rtx_description)/meshes/base_link.stl" scale="0.001 0.001 0.001"/>
+    </geometry>
+    <material name="silver"/>
+  </visual>
+  <collision>
+    <origin xyz="0 0 0" rpy="0 0 0"/>
+    <geometry>
+      <mesh filename="file://$(find dummy_rtx_description)/meshes/base_link.stl" scale="0.001 0.001 0.001"/>
+    </geometry>
+  </collision>
+</link>
 <link name="link1_1">
   <inertial>
@@ -42,5 +33,5 @@
     <origin xyz="-0.0 -0.0 -0.096" rpy="0 0 0"/>
     <geometry>
-      <mesh filename="file://$(find dummy_ros_r_description)/meshes/link1_1.stl" scale="0.001 0.001 0.001"/>
+      <mesh filename="file://$(find dummy_rtx_description)/meshes/link1_1.stl" scale="0.001 0.001 0.001"/>
     </geometry>
     <material name="silver"/>
@@ -49,5 +40,5 @@
     <origin xyz="-0.0 -0.0 -0.096" rpy="0 0 0"/>
     <geometry>
-      <mesh filename="file://$(find dummy_ros_r_description)/meshes/link1_1.stl" scale="0.001 0.001 0.001"/>
+      <mesh filename="file://$(find dummy_rtx_description)/meshes/link1_1.stl" scale="0.001 0.001 0.001"/>
     </geometry>
   </collision>
@@ -55,5 +46,5 @@
 <link name="link2_1">
   <inertial>
-    <origin xyz="0.01692171088136483 0.07109319413511461 0.019215100323449058" rpy="0 0 0"/>
+    <origin xyz="0.01692171088136483 0.07109319413511461 0.01921510032344903" rpy="0 0 0"/>
     <mass value="0.38848490516085693"/>
     <inertia ixx="0.001645" iyy="0.000269" izz="0.001568" ixy="0.000175" iyz="-0.000382" ixz="4.8e-05"/>
@@ -62,5 +53,5 @@
     <origin xyz="0.017 0.035 -0.1335" rpy="0 0 0"/>
     <geometry>
-      <mesh filename="file://$(find dummy_ros_r_description)/meshes/link2_1.stl" scale="0.001 0.001 0.001"/>
+      <mesh filename="file://$(find dummy_rtx_description)/meshes/link2_1.stl" scale="0.001 0.001 0.001"/>
     </geometry>
     <material name="silver"/>
@@ -69,5 +60,5 @@
     <origin xyz="0.017 0.035 -0.1335" rpy="0 0 0"/>
     <geometry>
-      <mesh filename="file://$(find dummy_ros_r_description)/meshes/link2_1.stl" scale="0.001 0.001 0.001"/>
+      <mesh filename="file://$(find dummy_rtx_description)/meshes/link2_1.stl" scale="0.001 0.001 0.001"/>
     </geometry>
   </collision>
@@ -75,5 +66,5 @@
 <link name="link3_1">
   <inertial>
-    <origin xyz="-0.01133047905022835 -0.00795343228580088 0.04187792038734822" rpy="0 0 0"/>
+    <origin xyz="-0.01133047905022835 -0.007953432285800852 0.04187792038734822" rpy="0 0 0"/>
     <mass value="0.23199545454229795"/>
     <inertia ixx="0.000142" iyy="0.000165" izz="8.9e-05" ixy="-6e-06" iyz="1.3e-05" ixz="3.8e-05"/>
@@ -82,5 +73,5 @@
     <origin xyz="-0.017 -0.106025 -0.171288" rpy="0 0 0"/>
     <geometry>
-      <mesh filename="file://$(find dummy_ros_r_description)/meshes/link3_1.stl" scale="0.001 0.001 0.001"/>
+      <mesh filename="file://$(find dummy_rtx_description)/meshes/link3_1.stl" scale="0.001 0.001 0.001"/>
     </geometry>
     <material name="silver"/>
@@ -89,5 +80,5 @@
     <origin xyz="-0.017 -0.106025 -0.171288" rpy="0 0 0"/>
     <geometry>
-      <mesh filename="file://$(find dummy_ros_r_description)/meshes/link3_1.stl" scale="0.001 0.001 0.001"/>
+      <mesh filename="file://$(find dummy_rtx_description)/meshes/link3_1.stl" scale="0.001 0.001 0.001"/>
     </geometry>
   </collision>
@@ -102,5 +93,5 @@
     <origin xyz="-0.0 -0.078561 -0.217763" rpy="0 0 0"/>
     <geometry>
-      <mesh filename="file://$(find dummy_ros_r_description)/meshes/link4_1.stl" scale="0.001 0.001 0.001"/>
+      <mesh filename="file://$(find dummy_rtx_description)/meshes/link4_1.stl" scale="0.001 0.001 0.001"/>
     </geometry>
     <material name="silver"/>
@@ -109,5 +100,5 @@
     <origin xyz="-0.0 -0.078561 -0.217763" rpy="0 0 0"/>
     <geometry>
-      <mesh filename="file://$(find dummy_ros_r_description)/meshes/link4_1.stl" scale="0.001 0.001 0.001"/>
+      <mesh filename="file://$(find dummy_rtx_description)/meshes/link4_1.stl" scale="0.001 0.001 0.001"/>
     </geometry>
   </collision>
@@ -115,5 +106,5 @@
 <link name="link5_1">
   <inertial>
-    <origin xyz="0.0009058322817682672 -0.028070035017605043 -0.007521517263662902" rpy="0 0 0"/>
+    <origin xyz="0.0009058322817682672 -0.028070035017605043 -0.007521517263662875" rpy="0 0 0"/>
     <mass value="0.04856312889395257"/>
     <inertia ixx="4.1e-05" iyy="1.4e-05" izz="4e-05" ixy="8e-06" iyz="-7e-06" ixz="2e-06"/>
@@ -122,5 +113,5 @@
     <origin xyz="0.0186 0.020447 -0.191234" rpy="0 0 0"/>
     <geometry>
-      <mesh filename="file://$(find dummy_ros_r_description)/meshes/link5_1.stl" scale="0.001 0.001 0.001"/>
+      <mesh filename="file://$(find dummy_rtx_description)/meshes/link5_1.stl" scale="0.001 0.001 0.001"/>
     </geometry>
     <material name="silver"/>
@@ -129,5 +120,5 @@
     <origin xyz="0.0186 0.020447 -0.191234" rpy="0 0 0"/>
     <geometry>
-      <mesh filename="file://$(find dummy_ros_r_description)/meshes/link5_1.stl" scale="0.001 0.001 0.001"/>
+      <mesh filename="file://$(find dummy_rtx_description)/meshes/link5_1.stl" scale="0.001 0.001 0.001"/>
     </geometry>
   </collision>
@@ -135,6 +126,6 @@
 <link name="link6_1">
   <inertial>
-    <origin xyz="1.4314084748695763e-05 -0.0024116315393477583 -0.0006596157012566661" rpy="0 0 0"/>
-    <mass value="0.020155987678957044"/>
+    <origin xyz="1.431408474869382e-05 -0.0024116315393478 -0.0006596157012566384" rpy="0 0 0"/>
+    <mass value="0.02015598767895705"/>
     <inertia ixx="1e-06" iyy="2e-06" izz="1e-06" ixy="0.0" iyz="0.0" ixz="-0.0"/>
   </inertial>
@@ -142,5 +133,5 @@
     <origin xyz="-0.0 0.080817 -0.175058" rpy="0 0 0"/>
     <geometry>
-      <mesh filename="file://$(find dummy_ros_r_description)/meshes/link6_1.stl" scale="0.001 0.001 0.001"/>
+      <mesh filename="file://$(find dummy_rtx_description)/meshes/link6_1.stl" scale="0.001 0.001 0.001"/>
     </geometry>
     <material name="silver"/>
@@ -149,5 +140,5 @@
     <origin xyz="-0.0 0.080817 -0.175058" rpy="0 0 0"/>
     <geometry>
-      <mesh filename="file://$(find dummy_ros_r_description)/meshes/link6_1.stl" scale="0.001 0.001 0.001"/>
+      <mesh filename="file://$(find dummy_rtx_description)/meshes/link6_1.stl" scale="0.001 0.001 0.001"/>
     </geometry>
   </collision>
@@ -158,5 +149,5 @@
   <child link="link1_1"/>
   <axis xyz="0.0 0.0 -1.0"/>
-  <limit upper="2.96706" lower="-2.96706" effort="100" velocity="100" acceleration="2.0"/>
+  <limit upper="2.96706" lower="-2.96706" effort="100" velocity="100"/>
 </joint>
 <joint name="Joint2" type="revolute">
@@ -165,5 +156,5 @@
   <child link="link2_1"/>
   <axis xyz="1.0 0.0 0.0"/>
-  <limit upper="2.879793" lower="0.0" effort="100" velocity="100" acceleration="2.0"/>
+  <limit upper="2.879793" lower="0.0" effort="100" velocity="100"/>
 </joint>
 <joint name="Joint3" type="revolute">
@@ -172,5 +163,5 @@
   <child link="link3_1"/>
   <axis xyz="-1.0 -0.0 -0.0"/>
-  <limit upper="3.752458" lower="0.0" effort="100" velocity="100" acceleration="2.0"/>
+  <limit upper="3.752458" lower="0.0" effort="100" velocity="100"/>
 </joint>
 <joint name="Joint4" type="revolute">
@@ -179,5 +170,5 @@
   <child link="link4_1"/>
   <axis xyz="-0.0 0.965926 0.258819"/>
-  <limit upper="3.141593" lower="0.0" effort="100" velocity="100" acceleration="2.0"/>
+  <limit upper="3.141593" lower="0.0" effort="100" velocity="100"/>
 </joint>
 <joint name="Joint5" type="revolute">
@@ -186,5 +177,5 @@
   <child link="link5_1"/>
   <axis xyz="-1.0 0.0 -0.0"/>
-  <limit upper="2.094395" lower="-2.094395" effort="100" velocity="100" acceleration="2.0"/>
+  <limit upper="2.094395" lower="-2.094395" effort="100" velocity="100"/>
 </joint>
 <joint name="Joint6" type="continuous">

File: src/dummy_rtx_moveit_config/config/dummy_ros_r.ros2_control.xacro (robot description, xacro)
@@ -2,5 +2,5 @@
 <robot xmlns:xacro="http://www.ros.org/wiki/xacro">
     <xacro:macro name="dummy_ros_r_ros2_control" params="name initial_positions_file">
-        <xacro:property name="initial_positions" value="${xacro.load_yaml(initial_positions_file)['initial_positions']}"/>
+        <xacro:property name="initial_positions" value="${load_yaml(initial_positions_file)['initial_positions']}"/>
         <ros2_control name="${name}" type="system">
             <hardware>

File: src/dummy_rtx_moveit_config/config/dummy_ros_r.urdf.xacro (robot description, xacro)
@@ -3,5 +3,5 @@
     <xacro:arg name="initial_positions_file" default="initial_positions.yaml" />
     <!-- Import dummy_ros_r urdf file -->
-    <xacro:include filename="$(find dummy_ros_r_description)/urdf/dummy_ros_r.xacro" />
+    <xacro:include filename="$(find dummy_rtx_description)/urdf/dummy_ros_r.xacro" />
     <!-- Import control_xacro -->
     <xacro:include filename="dummy_ros_r.ros2_control.xacro" />
