Commit message: modify description name

File: src/dummy_rtx_description/urdf/dummy_rtx.xacro (robot description, xacro)
@@ -1,7 +1,7 @@
 <?xml version="1.0" ?>
-<robot name="dummy_ros_r" xmlns:xacro="http://www.ros.org/wiki/xacro">
+<robot name="dummy_rtx" xmlns:xacro="http://www.ros.org/wiki/xacro">
 <xacro:include filename="$(find dummy_rtx_description)/urdf/materials.xacro" />
-<xacro:include filename="$(find dummy_rtx_description)/urdf/dummy_ros_r.trans" />
-<xacro:include filename="$(find dummy_rtx_description)/urdf/dummy_ros_r.gazebo" />
+<xacro:include filename="$(find dummy_rtx_description)/urdf/dummy_rtx.trans" />
+<xacro:include filename="$(find dummy_rtx_description)/urdf/dummy_rtx.gazebo" />
 <link name="base_link">
   <inertial>

File: src/dummy_rtx_description/urdf/materials.xacro (robot description, xacro)
@@ -1,4 +1,4 @@
 <?xml version="1.0" ?>
-<robot name="dummy_ros_r" xmlns:xacro="http://www.ros.org/wiki/xacro" >
+<robot name="dummy_rtx" xmlns:xacro="http://www.ros.org/wiki/xacro" >
 <material name="silver">
   <color rgba="0.700 0.700 0.700 1.000"/>

File: src/dummy_rtx_moveit_config/config/dummy_rtx.ros2_control.xacro (robot description, xacro)
@@ -1,5 +1,5 @@
 <?xml version="1.0"?>
 <robot xmlns:xacro="http://www.ros.org/wiki/xacro">
-    <xacro:macro name="dummy_ros_r_ros2_control" params="name initial_positions_file">
+    <xacro:macro name="dummy_rtx_ros2_control" params="name initial_positions_file">
         <xacro:property name="initial_positions" value="${load_yaml(initial_positions_file)['initial_positions']}"/>
         <ros2_control name="${name}" type="system">
